File: blink_board.kicad_pcb (KiCad board)
At the start: 4 copper layers, 85 x 55 mm, 25 parts, among them J1 USB_C_Receptacle_PowerOnly_6P, J2 Debug, SW1 BTN_1, SW2 BTN_2, U1 ESP-01v090, U2 MIC5504-3.3YM5, U3 MCP23017_SO

Commit message: Bugfixes and updates
* Added small board description
* Added testpads for I2C
* Fixed power for display
* Added labels for Serial
* Aligned buttons
* Cleaned silkscreen
Parts:
- added TP1: GND, TestPoint:TestPoint_Pad_D1.5mm, B.Cu at (112.3, 43.9)
- added TP2: SDA, TestPoint:TestPoint_Pad_D1.5mm, B.Cu at (117.3, 43.9)
- added TP3: SCL, TestPoint:TestPoint_Pad_D1.5mm, B.Cu at (114.8, 43.9)
- moved SW2 6.39 mm to (123.7, 52.0)
- moved R2 5.99 mm to (72.1, 42.9)
- moved SW1 5.76 mm to (123.7, 41.2)
Connections:
- Brd1 pad 1: GND -> +3V3
- Brd1 pad 2: +3V3 -> GND
Routing:
- net Net-(D1-K): track 9.87 -> 3.06 mm
- net Net-(SW2-B): track 34.8 -> 41.4 mm
- net Net-(SW1-B): track 50.2 -> 56.4 mm
- net Net-(U3-GPB0): track 73.3 -> 67.5 mm
- net /I2C_SDA: track 183.0 -> 181.5 mm
- net GND: track 221.8 -> 220.7 mm
- net +3V3: track 123.1 -> 122.1 mm
Other:
- board text added: "BLINK BOARD - V1.2"
- board text added: "TXD RXD GND"
